File: Eletrônica/Pontos Cegos - Rev A/Pontos Cegos - Rev A.brd (EAGLE design)
At the start: 60 x 60 mm, 37 parts, among them IC1 7806DT, J1 22-05-7028-02, U1 ATMEGA328P, X1 2510-, X2 2510-, Y1 16MHz

Commit message: BRD updated
Routing:
- net MOSI: track 39.1 -> 56.4 mm
- net D8: track 45.9 -> 47.7 mm
